File: matrix.kicad_sch (KiCad schematic)
At the start: 8 parts

Commit message: added keyswitch footprint submodule
Parts:
- D1, D2, D3, D4: footprint (none) -> Diode_SMD:D_SOD-123
Changed lines of the file:
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@@
 			)
 		)
-		(property "Footprint" ""
+		(property "Footprint" "Diode_SMD:D_SOD-123"
 			(at 93.98 91.44 0)
 			(effects
@@
 			)
 		)
-		(property "Footprint" ""
+		(property "Footprint" "Diode_SMD:D_SOD-123"
 			(at 93.98 72.39 0)
 			(effects
@@
 			)
 		)
-		(property "Footprint" ""
+		(property "Footprint" "Diode_SMD:D_SOD-123"
 			(at 132.08 91.44 0)
 			(effects
@@
 			)
 		)
-		(property "Footprint" ""
+		(property "Footprint" "Diode_SMD:D_SOD-123"
 			(at 132.08 72.39 0)
 			(effects

Commit message: WIP: footprints
Parts:
- KEY1, KEY2, KEY3, KEY4: footprint (none) -> MX_Hotswap:MX-Hotswap-1U
Changed lines of the file:
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@@
 			)
 		)
-		(property "Footprint" ""
+		(property "Footprint" "MX_Hotswap:MX-Hotswap-1U"
 			(at 85.09 82.55 0)
 			(effects
@@
 			)
 		)
-		(property "Footprint" ""
+		(property "Footprint" "MX_Hotswap:MX-Hotswap-1U"
 			(at 123.19 63.5 0)
 			(effects
@@
 			)
 		)
-		(property "Footprint" ""
+		(property "Footprint" "MX_Hotswap:MX-Hotswap-1U"
 			(at 123.19 82.55 0)
 			(effects
@@
 			)
 		)
-		(property "Footprint" ""
+		(property "Footprint" "MX_Hotswap:MX-Hotswap-1U"
 			(at 85.09 63.5 0)
 			(effects

Commit message: WIP:routing
Parts:
- added D10, D11, D12, D15, D16, D17, D18, D19, D20, D21, D22, D23, D24, D25, D26, D27, D28, D29, D3, D30, D31, D32, D33, D34, D35, D36, D37, D38, D39, D4, D40, D41, D42, D43, D44, D45, D46, D47, D48, D49, D5, D50, D51, D52, D53, D54, D55, D56, D57, D58, D59, D6, D60, D7, D8, D9: 1N4148W, Diode_SMD:D_SOD-123, symbol Device:D
- added KEY10, KEY11, KEY12, KEY15, KEY16, KEY17, KEY18, KEY19, KEY20, KEY21, KEY22, KEY23, KEY24, KEY25, KEY26, KEY27, KEY28, KEY29, KEY3, KEY30, KEY31, KEY32, KEY33, KEY34, KEY35, KEY36, KEY37, KEY38, KEY39, KEY4, KEY40, KEY41, KEY42, KEY43, KEY44, KEY45, KEY46, KEY47, KEY48, KEY49, KEY5, KEY50, KEY51, KEY52, KEY53, KEY54, KEY55, KEY56, KEY57, KEY58, KEY59, KEY6, KEY60, KEY7, KEY8, KEY9: MX_keyswitch, MX_Hotswap:MX-Hotswap-1U, symbol Switch:SW_Push
- renumbered D3 to D13, D4 to D14, KEY3 to KEY13, KEY4 to KEY14
Connections:
- net COL0: now also KEY25.1, KEY37.1, KEY49.1
- net COL1: now also KEY10.1, KEY11.1, KEY12.1, KEY15.1, KEY16.1, KEY17.1, KEY18.1, KEY19.1, KEY20.1, KEY21.1, KEY22.1, KEY23.1, KEY24.1, KEY26.1, KEY27.1, KEY28.1, KEY29.1, KEY3.1, KEY30.1, KEY31.1, KEY32.1, KEY33.1, KEY34.1, KEY35.1, KEY36.1, KEY38.1, KEY39.1, KEY4.1, KEY40.1, KEY41.1, KEY42.1, KEY43.1, KEY44.1, KEY45.1, KEY46.1, KEY47.1, KEY48.1, KEY5.1, KEY50.1, KEY51.1, KEY52.1, KEY53.1, KEY54.1, KEY55.1, KEY56.1, KEY57.1, KEY58.1, KEY59.1, KEY6.1, KEY60.1, KEY7.1, KEY8.1, KEY9.1
- net ROW0: now also D10.1 (K), D11.1 (K), D12.1 (K), D3.1 (K), D4.1 (K), D5.1 (K), D6.1 (K), D7.1 (K), D8.1 (K), D9.1 (K)
- net ROW1: now also D15.1 (K), D16.1 (K), D17.1 (K), D18.1 (K), D19.1 (K), D20.1 (K), D21.1 (K), D22.1 (K), D23.1 (K), D24.1 (K), D25.1 (K), D26.1 (K), D27.1 (K), D28.1 (K), D29.1 (K), D30.1 (K), D31.1 (K), D32.1 (K), D33.1 (K), D34.1 (K), D35.1 (K), D36.1 (K), D37.1 (K), D38.1 (K), D39.1 (K), D40.1 (K), D41.1 (K), D42.1 (K), D43.1 (K), D44.1 (K), D45.1 (K), D46.1 (K), D47.1 (K), D48.1 (K), D49.1 (K), D50.1 (K), D51.1 (K), D52.1 (K), D53.1 (K), D54.1 (K), D55.1 (K), D56.1 (K), D57.1 (K), D58.1 (K), D59.1 (K), D60.1 (K)
- new net: D8.2 (A), KEY8.2
- new net: D41.2 (A), KEY41.2
- new net: D9.2 (A), KEY9.2
- new net: D37.2 (A), KEY37.2
- new net: D3.2 (A), KEY3.2
- new net: D19.2 (A), KEY19.2
- new net: D24.2 (A), KEY24.2
- new net: D16.2 (A), KEY16.2
- new net: D43.2 (A), KEY43.2
- new net: D33.2 (A), KEY33.2
- new net: D47.2 (A), KEY47.2
- new net: D6.2 (A), KEY6.2
- new net: D12.2 (A), KEY12.2
- new net: D57.2 (A), KEY57.2
- new net: D48.2 (A), KEY48.2
- new net: D52.2 (A), KEY52.2
- new net: D22.2 (A), KEY22.2
- new net: D46.2 (A), KEY46.2
- new net: D30.2 (A), KEY30.2
- new net: D31.2 (A), KEY31.2
- new net: D25.2 (A), KEY25.2
- new net: D20.2 (A), KEY20.2
- new net: D23.2 (A), KEY23.2
- new net: D28.2 (A), KEY28.2
- new net: D35.2 (A), KEY35.2
- new net: D29.2 (A), KEY29.2
- new net: D10.2 (A), KEY10.2
- new net: D40.2 (A), KEY40.2
- new net: D55.2 (A), KEY55.2
- new net: D36.2 (A), KEY36.2
- new net: D60.2 (A), KEY60.2
- new net: D17.2 (A), KEY17.2
- new net: D50.2 (A), KEY50.2
- new net: D15.2 (A), KEY15.2
- new net: D26.2 (A), KEY26.2
- new net: D32.2 (A), KEY32.2
- new net: D44.2 (A), KEY44.2
- new net: D38.2 (A), KEY38.2
- new net: D51.2 (A), KEY51.2
- new net: D54.2 (A), KEY54.2
- new net: D11.2 (A), KEY11.2
- new net: D42.2 (A), KEY42.2
- new net: D7.2 (A), KEY7.2
- new net: D45.2 (A), KEY45.2
- new net: D53.2 (A), KEY53.2
- new net: D39.2 (A), KEY39.2
- new net: D59.2 (A), KEY59.2
- new net: D18.2 (A), KEY18.2
- new net: D4.2 (A), KEY4.2
- new net: D21.2 (A), KEY21.2
- new net: D49.2 (A), KEY49.2
- new net: D34.2 (A), KEY34.2
- new net: D5.2 (A), KEY5.2
- new net: D58.2 (A), KEY58.2
- new net: D27.2 (A), KEY27.2
- new net: D56.2 (A), KEY56.2
Other:
- moved on the sheet: D1, D13, D14, D2, KEY1, KEY13, KEY14, KEY2

Commit message: WIP: routed matrix and added swdio
Connections:
- net COL1: no longer KEY10.1, KEY11.1, KEY12.1, KEY15.1, KEY16.1, KEY17.1, KEY18.1, KEY19.1, KEY20.1, KEY21.1, KEY22.1, KEY23.1, KEY24.1, KEY27.1, KEY28.1, KEY29.1, KEY3.1, KEY30.1, KEY31.1, KEY32.1, KEY33.1, KEY34.1, KEY35.1, KEY36.1, KEY39.1, KEY4.1, KEY40.1, KEY41.1, KEY42.1, KEY43.1, KEY44.1, KEY45.1, KEY46.1, KEY47.1, KEY48.1, KEY5.1, KEY51.1, KEY52.1, KEY53.1, KEY54.1, KEY55.1, KEY56.1, KEY57.1, KEY58.1, KEY59.1, KEY6.1, KEY60.1, KEY7.1, KEY8.1, KEY9.1
- net ROW1: no longer D25.1 (K), D26.1 (K), D27.1 (K), D28.1 (K), D29.1 (K), D30.1 (K), D31.1 (K), D32.1 (K), D33.1 (K), D34.1 (K), D35.1 (K), D36.1 (K), D37.1 (K), D38.1 (K), D39.1 (K), D40.1 (K), D41.1 (K), D42.1 (K), D43.1 (K), D44.1 (K), D45.1 (K), D46.1 (K), D47.1 (K), D48.1 (K), D49.1 (K), D50.1 (K), D51.1 (K), D52.1 (K), D53.1 (K), D54.1 (K), D55.1 (K), D56.1 (K), D57.1 (K), D58.1 (K), D59.1 (K), D60.1 (K)
- net D_70: now reaches D8.2 (A), KEY8.2
- net D_43: now reaches D41.2 (A), KEY41.2
- net D_80: now reaches D9.2 (A), KEY9.2
- net D_03: now reaches D37.2 (A), KEY37.2
- net D_20: now reaches D3.2 (A), KEY3.2
- net D_61: now reaches D19.2 (A), KEY19.2
- net D_111: now reaches D24.2 (A), KEY24.2
- net D_31: now reaches D16.2 (A), KEY16.2
- net D_63: now reaches D43.2 (A), KEY43.2
- net D_82: now reaches D33.2 (A), KEY33.2
- net D_103: now reaches D47.2 (A), KEY47.2
- net D_50: now reaches D6.2 (A), KEY6.2
- net D_110: now reaches D12.2 (A), KEY12.2
- net D_84: now reaches D57.2 (A), KEY57.2
- net D_113: now reaches D48.2 (A), KEY48.2
- net D_34: now reaches D52.2 (A), KEY52.2
- net D_91: now reaches D22.2 (A), KEY22.2
- net D_93: now reaches D46.2 (A), KEY46.2
- net D_52: now reaches D30.2 (A), KEY30.2
- net D_62: now reaches D31.2 (A), KEY31.2
- net D_02: now reaches D25.2 (A), KEY25.2
- net D_71: now reaches D20.2 (A), KEY20.2
- net D_101: now reaches D23.2 (A), KEY23.2
- net D_32: now reaches D28.2 (A), KEY28.2
- net  D_102: now reaches D35.2 (A), KEY35.2
- net D_42: now reaches D29.2 (A), KEY29.2
- net D_90: now reaches D10.2 (A), KEY10.2
- net D_33: now reaches D40.2 (A), KEY40.2
- net D_64: now reaches D55.2 (A), KEY55.2
- net  D_112: now reaches D36.2 (A), KEY36.2
- net D_114: now reaches D60.2 (A), KEY60.2
- net D_01: now reaches D13.2 (A), KEY13.2
- net D_41: now reaches D17.2 (A), KEY17.2
- net D_14: now reaches D50.2 (A), KEY50.2
- net D_21: now reaches D15.2 (A), KEY15.2
- net D_12: now reaches D26.2 (A), KEY26.2
- net D_72: now reaches D32.2 (A), KEY32.2
- net D_73: now reaches D44.2 (A), KEY44.2
- net D_13: now reaches D38.2 (A), KEY38.2
- net D_24: now reaches D51.2 (A), KEY51.2
- net D_54: now reaches D54.2 (A), KEY54.2
- net D_100: now reaches D11.2 (A), KEY11.2
- net D_00: now reaches D1.2 (A), KEY1.2
- net D_53: now reaches D42.2 (A), KEY42.2
- net D_10: now reaches D2.2 (A), KEY2.2
- net D_60: now reaches D7.2 (A), KEY7.2
- net D_83: now reaches D45.2 (A), KEY45.2
- net D_44: now reaches D53.2 (A), KEY53.2
- net D_23: now reaches D39.2 (A), KEY39.2
- net D_104: now reaches D59.2 (A), KEY59.2
- net D_51: now reaches D18.2 (A), KEY18.2
- net D_11: now reaches D14.2 (A), KEY14.2
- net D_30: now reaches D4.2 (A), KEY4.2
- net D_81: now reaches D21.2 (A), KEY21.2
- net D_04: now reaches D49.2 (A), KEY49.2
- net  D_92: now reaches D34.2 (A), KEY34.2
- net D_40: now reaches D5.2 (A), KEY5.2
- net D_94: now reaches D58.2 (A), KEY58.2
- net D_22: now reaches D27.2 (A), KEY27.2
- net D_74: now reaches D56.2 (A), KEY56.2
- new net COL10: KEY11.1, KEY23.1, KEY35.1, KEY47.1, KEY59.1
- new net COL11: KEY12.1, KEY24.1, KEY36.1, KEY48.1, KEY60.1
- new net COL2: KEY15.1, KEY27.1, KEY3.1, KEY39.1, KEY51.1
- new net COL3: KEY16.1, KEY28.1, KEY4.1, KEY40.1, KEY52.1
- new net COL4: KEY17.1, KEY29.1, KEY41.1, KEY5.1, KEY53.1
- new net COL5: KEY18.1, KEY30.1, KEY42.1, KEY54.1, KEY6.1
- new net COL6: KEY19.1, KEY31.1, KEY43.1, KEY55.1, KEY7.1
- new net COL7: KEY20.1, KEY32.1, KEY44.1, KEY56.1, KEY8.1
- new net COL8: KEY21.1, KEY33.1, KEY45.1, KEY57.1, KEY9.1
- new net COL9: KEY10.1, KEY22.1, KEY34.1, KEY46.1, KEY58.1
- new net ROW2: D25.1 (K), D26.1 (K), D27.1 (K), D28.1 (K), D29.1 (K), D30.1 (K), D31.1 (K), D32.1 (K), D33.1 (K), D34.1 (K), D35.1 (K), D36.1 (K)
- new net ROW3: D37.1 (K), D38.1 (K), D39.1 (K), D40.1 (K), D41.1 (K), D42.1 (K), D43.1 (K), D44.1 (K), D45.1 (K), D46.1 (K), D47.1 (K), D48.1 (K)
- new net ROW4: D49.1 (K), D50.1 (K), D51.1 (K), D52.1 (K), D53.1 (K), D54.1 (K), D55.1 (K), D56.1 (K), D57.1 (K), D58.1 (K), D59.1 (K), D60.1 (K)
