File: uniboi.kicad_pcb (KiCad board)
At the start: 2 copper layers, 232.6 x 99.2 mm, 137 parts, among them J1 USB_C_Receptacle_USB2.0_16P, SW1 SW_Push, SW2 SW_SPDT, U1 STM32G0B1CBTx, U2 SRV05-4, U3 XC6206P332MR

Commit message: WIP: changed usb-c connector, updated schematics with the SRV05-4, updated routing
Parts:
- moved R2 5.78 mm to (249.0, 60.9)
- moved U2 1.96 mm to (245.5, 66.0), turned to -90 degrees
- moved C5 0.48 mm to (238.5, 83.1)
- moved SW1 0.48 mm to (230.6, 80.8)
- moved U1 0.48 mm to (241.0, 76.6)
- moved C3 0.37 mm to (241.0, 82.7)
- moved C4 0.37 mm to (241.0, 83.7)
- moved C1 0.32 mm to (243.1, 83.7)
- moved C2 0.32 mm to (243.1, 82.7)
- moved C6 0.12 mm to (250.6, 66.0)
Connections:
- U2 pad 1: unconnected-(U2-IO1-Pad1) -> D+
- U2 pad 6: unconnected-(U2-IO4-Pad6) -> D-
Routing:
- net Net-(J1-CC2): track 1.99 -> 12.1 mm, vias 0 -> 2
- net GND: track 1.78 -> 9.94 mm, vias 0 -> 13
- net D-: track 13.9 -> 19.7 mm, vias 0 -> 2
- net +5V: track 0.03 -> 5.43 mm
- net +3.3V: track 26.5 -> 31.1 mm
- net D+: track 13.9 -> 16.0 mm, vias 0 -> 2

Commit message: WIP: schematics and routing
Parts:
- J1: value USB_C_Receptacle_USB2.0_16P -> DX07S016JA3R1500; footprint Connector_USB:USB_C_Receptacle_HRO_TYPE-C-31-M-12 -> USB_C_rmerli:CONN12_DX07S_JAE
- moved R2 6.23 mm to (235.2, 58.9)
- moved U2 3.25 mm to (242.4, 65.2), turned to 0 degrees
- moved R1 1.73 mm to (249.3, 59.2), turned to 0 degrees
- moved F1 0.65 mm to (250.0, 63.0)
- moved J1 0.53 mm to (242.0, 57.8)
- renumbered C6 to C1, C7 to C2, C1 to C3, C2 to C4, C3 to C5, C4 to C6, C5 to C7, R2 to R1, R3 to R2, R1 to R3, U3 to U1, U1 to U3
Connections:
- R1 pad 1: Net-(J1-CC2) -> /CC2
- R2 pad 1: Net-(J1-CC1) -> /CC1
- U2 pad 1: D+ -> unconnected-(U2-IO1-Pad1)
- U2 pad 3: unconnected-(U2-IO2-Pad3) -> D-
- U2 pad 4: unconnected-(U2-IO3-Pad4) -> D+
- U2 pad 6: D- -> unconnected-(U2-IO4-Pad6)
Routing:
- net Net-(J1-CC2): track 12.1 -> 0.00 mm, vias 2 -> 0
- net /CC2: track 0.00 -> 6.85 mm
- net /CC1: track 0.00 -> 5.95 mm
- net D-: track 19.7 -> 15.0 mm
- net Net-(J1-CC1): track 4.03 -> 0.00 mm
- net VBUS: track 8.25 -> 9.88 mm, vias 0 -> 2
- net +5V: track 5.43 -> 6.95 mm
- net GND: track 9.94 -> 11.3 mm, vias 13 -> 16
- net D+: track 16.0 -> 17.2 mm
Other:
- board text added: "RST"

Commit message: WIP: routed matrix and added swdio
Parts:
- added J4: SW_pads, Connector:Tag-Connect_TC2030-IDC-NL_2x03_P1.27mm_Vertical, B.Cu at (246.2, 69.0)
- J1: footprint USB_C_rmerli:CONN12_DX07S_JAE -> USB_C_rmerli:CONN12_DX07S_JAE_no_edge_cuts
- U3: value STM32G0B1CBTx -> STM32G0B1CBT6
- moved D60 374.7 mm to (261.5, 142.5), turned to 90 degrees
- moved D48 368.2 mm to (261.5, 123.5), turned to 90 degrees
- moved D36 362.1 mm to (261.5, 104.5), turned to 90 degrees
- moved D59 356.1 mm to (242.5, 142.5), turned to 90 degrees
- moved D47 349.4 mm to (242.5, 123.5), turned to 90 degrees
- moved D12 344.4 mm to (256.4, 74.4), turned to 90 degrees
- moved D35 343.2 mm to (242.5, 104.5), turned to 90 degrees
- moved D58 337.5 mm to (223.5, 142.5), turned to 90 degrees
- moved D24 335.2 mm to (246.5, 94.5), turned to 0 degrees
- moved D46 330.6 mm to (223.5, 123.5), turned to 90 degrees
- moved D34 319.2 mm to (223.5, 104.5), turned to 90 degrees
- moved D57 318.9 mm to (204.5, 142.5), turned to 90 degrees
- moved D11 317.3 mm to (226.4, 66.5), turned to 90 degrees
- moved D23 314.5 mm to (225.5, 92.5), turned to 90 degrees
- moved D22 313.5 mm to (223.5, 85.5), turned to 90 degrees
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Connections:
- net Net-(D1-A) renamed /matrix/D_00
- net Net-(D10-A) renamed /matrix/D_90
- net Net-(D11-A) renamed /matrix/D_100
- net Net-(D12-A) renamed /matrix/D_110
- net Net-(D13-A) renamed /matrix/D_01
- net Net-(D14-A) renamed /matrix/D_11
- net Net-(D15-A) renamed /matrix/D_21
- net Net-(D16-A) renamed /matrix/D_31
- net Net-(D17-A) renamed /matrix/D_41
- net Net-(D18-A) renamed /matrix/D_51
- net Net-(D19-A) renamed /matrix/D_61
- net Net-(D2-A) renamed /matrix/D_10
- net Net-(D20-A) renamed /matrix/D_71
- net Net-(D21-A) renamed /matrix/D_81
- net Net-(D22-A) renamed /matrix/D_91
- net Net-(D23-A) renamed /matrix/D_101
- net Net-(D24-A) renamed /matrix/D_111
- net Net-(D25-A) renamed /matrix/D_02
- net Net-(D26-A) renamed /matrix/D_12
- net Net-(D27-A) renamed /matrix/D_22
- net Net-(D28-A) renamed /matrix/D_32
- net Net-(D29-A) renamed /matrix/D_42
- net Net-(D3-A) renamed /matrix/D_20
- net Net-(D30-A) renamed /matrix/D_52
- net Net-(D31-A) renamed /matrix/D_62
- net Net-(D32-A) renamed /matrix/D_72
- net Net-(D33-A) renamed /matrix/D_82
- net Net-(D34-A) renamed /matrix/ D_92
- net Net-(D35-A) renamed /matrix/ D_102
- net Net-(D36-A) renamed /matrix/ D_112
- net Net-(D37-A) renamed /matrix/D_03
- net Net-(D38-A) renamed /matrix/D_13
- net Net-(D39-A) renamed /matrix/D_23
- net Net-(D4-A) renamed /matrix/D_30
- net Net-(D40-A) renamed /matrix/D_33
- net Net-(D41-A) renamed /matrix/D_43
- net Net-(D42-A) renamed /matrix/D_53
- net Net-(D43-A) renamed /matrix/D_63
- net Net-(D44-A) renamed /matrix/D_73
- net Net-(D45-A) renamed /matrix/D_83
- net Net-(D46-A) renamed /matrix/D_93
- net Net-(D47-A) renamed /matrix/D_103
- net Net-(D48-A) renamed /matrix/D_113
- net Net-(D49-A) renamed /matrix/D_04
- net Net-(D5-A) renamed /matrix/D_40
- net Net-(D50-A) renamed /matrix/D_14
- net Net-(D51-A) renamed /matrix/D_24
- net Net-(D52-A) renamed /matrix/D_34
- net Net-(D53-A) renamed /matrix/D_44
- net Net-(D54-A) renamed /matrix/D_54
- net Net-(D55-A) renamed /matrix/D_64
- net Net-(D56-A) renamed /matrix/D_74
- net Net-(D57-A) renamed /matrix/D_84
- net Net-(D58-A) renamed /matrix/D_94
- net Net-(D59-A) renamed /matrix/D_104
- net Net-(D6-A) renamed /matrix/D_50
- net Net-(D60-A) renamed /matrix/D_114
- net Net-(D7-A) renamed /matrix/D_60
- net Net-(D8-A) renamed /matrix/D_70
- net Net-(D9-A) renamed /matrix/D_80
- D1 pad 1: /matrix/ROW0 -> ROW0
- D10 pad 1: /matrix/ROW0 -> ROW0
- D11 pad 1: /matrix/ROW0 -> ROW0
- D12 pad 1: /matrix/ROW0 -> ROW0
- D13 pad 1: /matrix/ROW1 -> ROW1
- D14 pad 1: /matrix/ROW1 -> ROW1
- D15 pad 1: /matrix/ROW1 -> ROW1
- D16 pad 1: /matrix/ROW1 -> ROW1
- D17 pad 1: /matrix/ROW1 -> ROW1
- D18 pad 1: /matrix/ROW1 -> ROW1
- D19 pad 1: /matrix/ROW1 -> ROW1
- D2 pad 1: /matrix/ROW0 -> ROW0
- D20 pad 1: /matrix/ROW1 -> ROW1
- D21 pad 1: /matrix/ROW1 -> ROW1
- D22 pad 1: /matrix/ROW1 -> ROW1
- D23 pad 1: /matrix/ROW1 -> ROW1
- D24 pad 1: /matrix/ROW1 -> ROW1
- D25 pad 1: /matrix/ROW1 -> ROW2
- D26 pad 1: /matrix/ROW1 -> ROW2
- D27 pad 1: /matrix/ROW1 -> ROW2
- D28 pad 1: /matrix/ROW1 -> ROW2
- D29 pad 1: /matrix/ROW1 -> ROW2
- D3 pad 1: /matrix/ROW0 -> ROW0
- D30 pad 1: /matrix/ROW1 -> ROW2
- D31 pad 1: /matrix/ROW1 -> ROW2
- D32 pad 1: /matrix/ROW1 -> ROW2
- D33 pad 1: /matrix/ROW1 -> ROW2
- D34 pad 1: /matrix/ROW1 -> ROW2
- D35 pad 1: /matrix/ROW1 -> ROW2
- D36 pad 1: /matrix/ROW1 -> ROW2
- D37 pad 1: /matrix/ROW1 -> ROW3
- D38 pad 1: /matrix/ROW1 -> ROW3
- D39 pad 1: /matrix/ROW1 -> ROW3
- D4 pad 1: /matrix/ROW0 -> ROW0
- D40 pad 1: /matrix/ROW1 -> ROW3
- D41 pad 1: /matrix/ROW1 -> ROW3
- D42 pad 1: /matrix/ROW1 -> ROW3
- D43 pad 1: /matrix/ROW1 -> ROW3
- D44 pad 1: /matrix/ROW1 -> ROW3
- D45 pad 1: /matrix/ROW1 -> ROW3
- D46 pad 1: /matrix/ROW1 -> ROW3
- D47 pad 1: /matrix/ROW1 -> ROW3
- D48 pad 1: /matrix/ROW1 -> ROW3
- D49 pad 1: /matrix/ROW1 -> ROW4
- D5 pad 1: /matrix/ROW0 -> ROW0
- D50 pad 1: /matrix/ROW1 -> ROW4
- D51 pad 1: /matrix/ROW1 -> ROW4
- D52 pad 1: /matrix/ROW1 -> ROW4
- D53 pad 1: /matrix/ROW1 -> ROW4
- D54 pad 1: /matrix/ROW1 -> ROW4
- D55 pad 1: /matrix/ROW1 -> ROW4
- D56 pad 1: /matrix/ROW1 -> ROW4
- D57 pad 1: /matrix/ROW1 -> ROW4
- D58 pad 1: /matrix/ROW1 -> ROW4
- D59 pad 1: /matrix/ROW1 -> ROW4
- D6 pad 1: /matrix/ROW0 -> ROW0
- D60 pad 1: /matrix/ROW1 -> ROW4
- D7 pad 1: /matrix/ROW0 -> ROW0
- D8 pad 1: /matrix/ROW0 -> ROW0
- D9 pad 1: /matrix/ROW0 -> ROW0
- KEY10 pad 1: COL1 -> COL9
- KEY11 pad 1: COL1 -> COL10
- KEY12 pad 1: COL1 -> COL11
- KEY15 pad 1: COL1 -> COL2
- KEY16 pad 1: COL1 -> COL3
- KEY17 pad 1: COL1 -> COL4
- KEY18 pad 1: COL1 -> COL5
- KEY19 pad 1: COL1 -> COL6
- KEY20 pad 1: COL1 -> COL7
- KEY21 pad 1: COL1 -> COL8
- KEY22 pad 1: COL1 -> COL9
- KEY23 pad 1: COL1 -> COL10
- KEY24 pad 1: COL1 -> COL11
- KEY27 pad 1: COL1 -> COL2
- KEY28 pad 1: COL1 -> COL3
- KEY29 pad 1: COL1 -> COL4
- KEY3 pad 1: COL1 -> COL2
- KEY30 pad 1: COL1 -> COL5
- KEY31 pad 1: COL1 -> COL6
- KEY32 pad 1: COL1 -> COL7
- KEY33 pad 1: COL1 -> COL8
- KEY34 pad 1: COL1 -> COL9
- KEY35 pad 1: COL1 -> COL10
- KEY36 pad 1: COL1 -> COL11
- KEY39 pad 1: COL1 -> COL2
- KEY4 pad 1: COL1 -> COL3
- KEY40 pad 1: COL1 -> COL3
- KEY41 pad 1: COL1 -> COL4
- KEY42 pad 1: COL1 -> COL5
- KEY43 pad 1: COL1 -> COL6
- KEY44 pad 1: COL1 -> COL7
- KEY45 pad 1: COL1 -> COL8
- KEY46 pad 1: COL1 -> COL9
- KEY47 pad 1: COL1 -> COL10
- KEY48 pad 1: COL1 -> COL11
- KEY5 pad 1: COL1 -> COL4
- KEY51 pad 1: COL1 -> COL2
- KEY52 pad 1: COL1 -> COL3
- KEY53 pad 1: COL1 -> COL4
- KEY54 pad 1: COL1 -> COL5
- KEY55 pad 1: COL1 -> COL6
- KEY56 pad 1: COL1 -> COL7
- KEY57 pad 1: COL1 -> COL8
- KEY58 pad 1: COL1 -> COL9
- KEY59 pad 1: COL1 -> COL10
- KEY6 pad 1: COL1 -> COL5
- KEY60 pad 1: COL1 -> COL11
- KEY7 pad 1: COL1 -> COL6
- KEY8 pad 1: COL1 -> COL7
- KEY9 pad 1: COL1 -> COL8
- U3 pad 12: unconnected-(U3-PA1-Pad12) -> COL0
- U3 pad 13: unconnected-(U3-PA2-Pad13) -> COL1
- U3 pad 14: unconnected-(U3-PA3-Pad14) -> COL2
- U3 pad 15: unconnected-(U3-PA4-Pad15) -> COL3
- U3 pad 16: unconnected-(U3-PA5-Pad16) -> COL4
- U3 pad 17: unconnected-(U3-PA6-Pad17) -> COL5
- U3 pad 18: unconnected-(U3-PA7-Pad18) -> COL6
- U3 pad 19: unconnected-(U3-PB0-Pad19) -> COL7
- U3 pad 20: unconnected-(U3-PB1-Pad20) -> COL8
- U3 pad 21: unconnected-(U3-PB2-Pad21) -> COL9
- U3 pad 22: unconnected-(U3-PB10-Pad22) -> COL10
- U3 pad 35: unconnected-(U3-PA13-Pad35) -> SWDIO
- U3 pad 37: unconnected-(U3-PA15-Pad37) -> ROW0
- U3 pad 42: unconnected-(U3-PB3-Pad42) -> COL11
- U3 pad 43: unconnected-(U3-PB4-Pad43) -> ROW4
- U3 pad 45: unconnected-(U3-PB6-Pad45) -> ROW3
- U3 pad 47: COL1 -> ROW2
- U3 pad 48: COL0 -> ROW1
Routing:
- net ROW4: track 0.00 -> 303.6 mm, vias 0 -> 13
- net COL0: track 0.00 -> 282.1 mm, vias 0 -> 2
- net ROW3: track 0.00 -> 278.9 mm, vias 0 -> 15
- net COL1: track 0.00 -> 260.1 mm, vias 0 -> 2
- net ROW2: track 0.00 -> 257.8 mm, vias 0 -> 13
- net COL2: track 0.00 -> 240.8 mm, vias 0 -> 2
- net ROW1: track 0.00 -> 230.5 mm, vias 0 -> 13
- net ROW0: track 0.00 -> 222.8 mm, vias 0 -> 13
- net COL3: track 0.00 -> 221.6 mm, vias 0 -> 2
- net COL4: track 0.00 -> 202.3 mm, vias 0 -> 2
- net COL5: track 0.00 -> 183.0 mm, vias 0 -> 2
- net COL6: track 0.00 -> 163.8 mm, vias 0 -> 2
- net COL7: track 0.00 -> 144.6 mm, vias 0 -> 2
- net COL8: track 0.00 -> 125.6 mm, vias 0 -> 2
- net COL11: track 0.00 -> 114.1 mm, vias 0 -> 3
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
Commit message: WIP: updated usb VBUS route
Routing:
- net VBUS: track 9.88 -> 5.87 mm
Changed lines of the file:
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@@
 	)
 	(segment
-		(start 239.57738 62.194411)
-		(end 239.57738 60.550098)
-		(width 0.5)
+		(start 239.59 62.24)
+		(end 244.27 62.24)
+		(width 0.6)
 		(layer "F.Cu")
 		(net 7)
 	)
 	(segment
-		(start 240.933067 59.194411)
-		(end 242.933067 59.194411)
-		(width 0.5)
-		(layer "F.Cu")
-		(net 7)
-	)
-	(segment
-		(start 242.933067 59.194411)
-		(end 244.327835 60.589179)
-		(width 0.5)
-		(layer "F.Cu")
-		(net 7)
-	)
-	(segment
-		(start 239.57738 60.550098)
-		(end 240.933067 59.194411)
-		(width 0.5)
-		(layer "F.Cu")
-		(net 7)
-	)
-	(segment
-		(start 244.327835 60.589179)
-		(end 244.327835 61.79692)
+		(start 244.27 62.24)
+		(end 244.28 62.23)
 		(width 0.5)
 		(layer "F.Cu")
@@
 	)
 	(via
-		(at 239.57738 62.194411)
+		(at 239.59 62.24)
 		(size 0.6)
 		(drill 0.3)
@@
 	)
 	(via
-		(at 244.327835 61.79692)
+		(at 244.28 62.23)
 		(size 0.6)
 		(drill 0.3)
@@
 	)
 	(segment
-		(start 239.59 62.181791)
-		(end 239.57738 62.194411)
+		(start 239.59 62.24)
+		(end 239.59 61.06)
 		(width 0.5)
 		(layer "B.Cu")
-		(net 7)
-	)
-	(segment
-		(start 239.59 61.06)
-		(end 239.59 62.181791)
-		(width 0.5)
-		(layer "B.Cu")

Commit message: clean up and final touches
Parts:
- added REF**: MountingHole_2.2mm_M2_DIN965_Pad_TopBottom, MountingHole:MountingHole_2.2mm_M2_DIN965_Pad_TopBottom, F.Cu at (36.4, 150.8)
- added REF**: MountingHole_2.2mm_M2_DIN965_Pad_TopBottom, MountingHole:MountingHole_2.2mm_M2_DIN965_Pad_TopBottom, F.Cu at (36.4, 58.4)
- added REF**: MountingHole_2.2mm_M2_DIN965_Pad_TopBottom, MountingHole:MountingHole_2.2mm_M2_DIN965_Pad_TopBottom, F.Cu at (262.2, 58.4)
- added REF**: MountingHole_2.2mm_M2_DIN965_Pad_TopBottom, MountingHole:MountingHole_2.2mm_M2_DIN965_Pad_TopBottom, F.Cu at (262.2, 150.8)
- moved R1 0.43 mm to (249.4, 58.8)
Routing:
- net +3.3V: track 47.8 -> 43.6 mm
- net GND: track 11.3 -> 12.9 mm, vias 17 -> 139
- net ROW4: track 303.6 -> 304.9 mm
- net VBUS: track 5.87 -> 7.10 mm
- net ROW3: track 278.9 -> 279.9 mm
- net COL11: track 114.1 -> 115.1 mm
- net ROW1: track 230.5 -> 229.9 mm
- added copper zone on B.Cu, net +3.3V
Other:
- board text added: "09-04-2026"
- board text added: "1 A"
- board text added: "3"
- board text added: "G"
- board text added: "R"
- board text added: "RM 04/26 V1 Rev A"
- board text added: "S"
- board text added: "Uniboi"
- board text added: "Uniboi kb"
