File: uniboi.kicad_pcb (KiCad board)
At the start: 2 copper layers, 232.6 x 99.2 mm, 142 parts, among them J1 DX07S016JA3R1500, J4 SW_pads, SW1 SW_Push, SW2 SW_SPDT, U1 XC6206P332MR, U2 SRV05-4, U3 STM32G0B1CBT6

Commit message: clean up and final touches
Parts:
- J4: footprint Connector:Tag-Connect_TC2030-IDC-NL_2x03_P1.27mm_Vertical -> connector:Tag-Connect_TC2030-IDC-NL_2x03_P1.27mm_Vertical
Changed lines of the file:
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@@
 			(net 2 "GND")
 			(pinfunction "GND")
-			(pintype "power_out")
+			(pintype "power_in")
 		)
 		(pad "2" smd rect
@@
 			(net 2 "GND")
 			(pinfunction "GND")
-			(pintype "power_out")
+			(pintype "power_in")
 		)
 		(pad "17" smd rect
@@
 		)
 	)
-	(footprint "Connector:Tag-Connect_TC2030-IDC-NL_2x03_P1.27mm_Vertical"
+	(footprint "connector:Tag-Connect_TC2030-IDC-NL_2x03_P1.27mm_Vertical"
 		(layer "B.Cu")
 		(at 246.2 69 90)
@@
 		(tags "tag connect programming header pogo pins")
 		(property "Reference" "J4"
-			(at 0 -2.7 90)
+			(at 0 -2.7 270)
 			(layer "B.SilkS")
-			(hide yes)
 			(effects
 				(font
@@
 		)
 		(property "Value" "SW_pads"
-			(at 0 2.3 90)
+			(at 0 2.3 270)
 			(layer "B.Fab")
 			(effects
@@
 			(layer "B.CrtYd")
 		)
-		(fp_text user "KEEPOUT"
-			(at 0 0 90)
-			(layer "Cmts.User")
-			(effects
-				(font
-					(size 0.4 0.4)
-					(thickness 0.07)
-				)
-			)
-		)
 		(fp_text user "${REFERENCE}"
-			(at 0 0 90)
+			(at 0 0 270)
 			(layer "B.Fab")
 			(effects
@@
 	)
 	(segment
-		(start 243.135 69.04)
-		(end 244.45 67.725)
+		(start 236.075 80.325)
+		(end 236.075 72.935)
 		(width 0.2)
 		(layer "F.Cu")
@@
 	)
 	(segment
-		(start 236.075 80.325)
-		(end 236.075 72.675)
+		(start 243.135 69.04)
+		(end 244.45 67.725)
 		(width 0.2)
 		(layer "F.Cu")
@@
 	)
 	(segment
-		(start 234.5 81.9)
-		(end 236.075 80.325)
+		(start 239.97 69.04)
+		(end 243.135 69.04)
 		(width 0.2)
 		(layer "F.Cu")
@@
 	)
 	(segment
-		(start 236.075 72.675)
-		(end 239.71 69.04)
+		(start 236.075 72.935)
+		(end 239.97 69.04)
 		(width 0.2)
 		(layer "F.Cu")
@@
 	)
 	(segment
-		(start 239.71 69.04)
-		(end 243.135 69.04)
+		(start 234.5 81.9)
+		(end 236.075 80.325)
 		(width 0.2)
 		(layer "F.Cu")
